Commit message: half tested create_config.sh and created config files for all 3 objects, world files have been created sans objects

File: models/home_floor_plan/urdf/home_floor_plan.urdf (robot description, URDF)
Before this commit: robot Home Floor plan, 1 links, 0 joints
Links:
- removed link Home
- added link home_floor_plan, mass 23856; collision mesh filename=package://home_floor_plan/meshes/home_floor_plan.STL; visual mesh filename=package://home_floor_plan/meshes/home_floor_plan.STL

File: models/linnmon_table/urdf/linnmon_table.urdf (robot description, URDF)
Before this commit: robot Ikea Linnmon, 1 links, 0 joints
Links:
- removed link Ikea Linnmon
- added link linnmon_table, mass 23.919; collision mesh filename=package://linnmon_table/meshes/linnmon_table.STL; visual mesh filename=package://linnmon_table/meshes/linnmon_table.STL
